Commit message: a working version of isaac and moveit piper

File: piper_camera_moveit_config/config/piper_description.ros2_control.xacro (robot description, xacro)
@@ -1,14 +1,17 @@
 <?xml version="1.0"?>
 <robot xmlns:xacro="http://www.ros.org/wiki/xacro">
-    <xacro:macro name="piper_description_ros2_control" params="name initial_positions_file">
-        <xacro:property name="initial_positions" value="${load_yaml(initial_positions_file)['initial_positions']}"/>
-        <ros2_control name="${name}" type="system">
-            <hardware>
-                <!-- By default, set up controllers for simulation. This won't work on real hardware -->
-                <!-- <plugin>mock_components/GenericSystem</plugin> -->
+  <xacro:macro name="piper_description_ros2_control" params="name initial_positions_file ros2_control_hardware_type:=mock_components">
+      <xacro:property name="initial_positions" value="${load_yaml(initial_positions_file)['initial_positions']}"/>
+      <ros2_control name="${name}" type="system">
+          <hardware>
+            <xacro:if value="${ros2_control_hardware_type == 'mock_components'}">
+                <plugin>mock_components/GenericSystem</plugin>
+            </xacro:if>
+            <xacro:if value="${ros2_control_hardware_type == 'isaac'}">
                 <plugin>topic_based_ros2_control/TopicBasedSystem</plugin>
                 <param name="joint_commands_topic">/isaac_joint_commands</param>
                 <param name="joint_states_topic">/isaac_joint_states</param>
-            </hardware>
+            </xacro:if>
+          </hardware>
             <joint name="joint1">
                 <command_interface name="position"/>

File: piper_camera_moveit_config/config/piper_description.urdf.xacro (robot description, xacro)
@@ -2,8 +2,9 @@
 <robot xmlns:xacro="http://www.ros.org/wiki/xacro" name="piper_description">
     <xacro:arg name="initial_positions_file" default="initial_positions.yaml" />
+    <xacro:arg name="ros2_control_hardware_type" default="mock_components" />
     <!-- Import piper_description urdf file -->
     <xacro:include filename="$(find piper_description)/urdf/piper_description.urdf" />
     <!-- Import control_xacro -->
     <xacro:include filename="piper_description.ros2_control.xacro" />
-    <xacro:piper_description_ros2_control name="FakeSystem" initial_positions_file="$(arg initial_positions_file)"/>
+    <xacro:piper_description_ros2_control name="FakeSystem" initial_positions_file="$(arg initial_positions_file)" ros2_control_hardware_type="$(arg ros2_control_hardware_type)"/>
 </robot>
